File: hardware/Macro_Keyboard_V1.1/Macro_Keyboard_V1.1.kicad_pcb (KiCad board)
At the start: 2 copper layers, 91.4 x 67.1 mm, 35 parts, among them SW1 Cherry MX, SW10 SW_Push, SW11 SW_Push, SW12 SW_Push, SW13 SW_SPDT, SW2 Cherry MX, SW3 Cherry MX, SW4 Cherry MX, SW5 Cherry MX, SW6 Cherry MX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

Commit message: Added 3d models for all components
Parts:
- SW10, SW11, SW12: footprint Button_Switch_THT:SW_PUSH_6mm_H5mm -> Macro-Keyboard-footprints:SW_PUSH_6mm_H7.3mm
