File: hardware/Macro_Keyboard_V1.1/Macro_Keyboard_V1.1.kicad_sch (KiCad schematic)
At the start: 29 parts, among them SW1 Cherry MX, SW10 SW_Push, SW11 SW_Push, SW12 SW_Push, SW13 SW_SPDT, SW2 Cherry MX, SW3 Cherry MX, SW4 Cherry MX, SW5 Cherry MX, SW6 Cherry MX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

Commit message: Added 3d models for all components
Parts:
- SW10, SW11, SW12: footprint Button_Switch_THT:SW_PUSH_6mm_H5mm -> Macro-Keyboard-footprints:SW_PUSH_6mm_H7.3mm
Changed lines of the file:
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@@
       (effects (font (size 1.27 1.27)) (justify right))
     )
-    (property "Footprint" "Button_Switch_THT:SW_PUSH_6mm_H5mm" (id 2) (at 219.456 131.318 0)
+    (property "Footprint" "Macro-Keyboard-footprints:SW_PUSH_6mm_H7.3mm" (id 2) (at 219.456 131.318 0)
       (effects (font (size 1.27 1.27)) hide)
     )
@@
       (effects (font (size 1.27 1.27)) (justify right))
     )
-    (property "Footprint" "Button_Switch_THT:SW_PUSH_6mm_H5mm" (id 2) (at 199.136 131.318 0)
+    (property "Footprint" "Macro-Keyboard-footprints:SW_PUSH_6mm_H7.3mm" (id 2) (at 199.136 131.318 0)
       (effects (font (size 1.27 1.27)) hide)
     )
@@
       (effects (font (size 1.27 1.27)) (justify right))
     )
-    (property "Footprint" "Button_Switch_THT:SW_PUSH_6mm_H5mm" (id 2) (at 178.816 131.318 0)
+    (property "Footprint" "Macro-Keyboard-footprints:SW_PUSH_6mm_H7.3mm" (id 2) (at 178.816 131.318 0)
       (effects (font (size 1.27 1.27)) hide)
     )
@@
     )
     (path "/decd62d9-b505-402b-86c5-efa565c0a450"
-      (reference "SW10") (unit 1) (value "SW_Push") (footprint "Button_Switch_THT:SW_PUSH_6mm_H5mm")
+      (reference "SW10") (unit 1) (value "SW_Push") (footprint "Macro-Keyboard-footprints:SW_PUSH_6mm_H7.3mm")
     )
     (path "/1faca474-e7d4-4d2f-af5f-3d9e5135f195"
-      (reference "SW11") (unit 1) (value "SW_Push") (footprint "Button_Switch_THT:SW_PUSH_6mm_H5mm")
+      (reference "SW11") (unit 1) (value "SW_Push") (footprint "Macro-Keyboard-footprints:SW_PUSH_6mm_H7.3mm")
     )
     (path "/14783d61-38c3-4b25-9775-53ff0f1543c9"
-      (reference "SW12") (unit 1) (value "SW_Push") (footprint "Button_Switch_THT:SW_PUSH_6mm_H5mm")
+      (reference "SW12") (unit 1) (value "SW_Push") (footprint "Macro-Keyboard-footprints:SW_PUSH_6mm_H7.3mm")
     )
     (path "/cc8ba0ca-9a72-4286-909d-907320468d1e"
